File: Hardware/PCB/asd.kicad_sch (KiCad schematic)
At the start: 68 parts, among them J1 za_motor_1, J10 dovod1, J11 dovod2, J12 extra masa, J13 Conn_01x06_Pin, J14 Stikalo3, J15 Za_stikalo, J16 Za_stikalo, J17 Za_stikalo, J18 Stikalo3, J19 Screw_Terminal_01x02, J2 za_motor_1, J20 Screw_Terminal_01x02, J21 Screw_Terminal_01x02, J22 Stikalo3, J23 Conn_01x08_Pin, J24 Conn_01x06_Pin, J25 Conn_01x10_Pin, J26 Conn_01x08_Pin, J27 napajanje STM32, J3 za_motor_1, J4 za_motor_2, J5 za_motor_2, J6 za_motor_2, J7 za_motor_3, J8 za_motor_3, J9 za_motor_3, Q1 2SC5566-TD-E, Q2 2SC5566-TD-E, Q3 2SC5566-TD-E, Q4 2SC5566-TD-E, Q5 2SC5566-TD-E, Q6 2SC5566-TD-E

Commit message: Add files via upload
Other:
- note added: "---------------------------------"
- note added: "= DC DIR"
- note added: "= DC PU"
- note added: "= M1 DIR"
- note added: "= M1 PU"
- note added: "= M1 SW"
- note added: "= M2 DIR"
- note added: "= M2 PU"
- note added: "= M2 SW"
- note added: "= M3 DIR"
- note added: "= M3 PU"
- note added: "= M3 SW"
- note added: "= M4 DIR"
- note added: "= M4 PU"
- note added: "= MANUAL SW1"
- note added: "= MANUAL SW2"
- note added: "= MANUAL SW3"
- note added: "DC SW1 ="
- note added: "DC SW2 ="
- note added: "PRITISK SENZOR ="
- note added: "TOF SCL ="
- note added: "TOF SDA ="
